Commit message: WIP: got to visuzlize in rviz! yay!

File: src/anymal_c_twins/urdf/leg/foot/foot_3_1_1_macro.urdf.xacro (robot description, xacro)
@@ -1,5 +1,5 @@
 <?xml version="1.0"?>
 <robot xmlns:xacro="http://www.ros.org/wiki/xacro">
-  <xacro:macro name="anymal_foot" params="leg:=LF">
+  <xacro:macro name="anymal_foot" params="leg:=LF suffix:='A'">
     <xacro:property name="S_r_SF_x"               value="0.087950"/> <!-- [m] -->
     <xacro:property name="S_r_SF_y"               value="0.013050"/> <!-- [m] -->
@@ -34,17 +34,17 @@
     </xacro:if>
     <!-- joint shank foot -->
-    <joint name="${leg}_shank_fixed_${leg}_FOOT" type="fixed">
-      <parent link="${leg}_shank_fixed"/>
-      <child link="${leg}_FOOT"/>
+    <joint name="${leg}_shank_fixed_${leg}_FOOT_${suffix}" type="fixed">
+      <parent link="${leg}_shank_fixed_${suffix}"/>
+      <child link="${leg}_FOOT_${suffix}"/>
       <origin xyz="${front*S_r_SF_x} ${left*S_r_SF_y} ${S_r_SF_z}"
               rpy="0 0 0"/>
     </joint>
     <!-- Foot link -->
-    <link name="${leg}_FOOT">
+    <link name="${leg}_FOOT_${suffix}">
      <visual>
        <origin xyz="0 0 0" rpy="0 0 ${(front-1)*0.5*pi - (front*left*pi*0.25)}"/>
        <geometry>
          <mesh
-             filename="package://anymal_c/urdf/leg/foot/foot_3_1_1_mesh.dae"
+             filename="package://anymal_c_twins/urdf/leg/foot/foot_3_1_1_mesh.dae"
              scale="${anymal_meshes_scale}"/>
        </geometry>
@@ -73,5 +73,5 @@
     </link>
     <!-- Gazebo customization -->
-    <gazebo reference="${leg}_FOOT">
+    <gazebo reference="${leg}_FOOT_${suffix}">
       <kp>${kp}</kp>
       <kd>${kd}</kd>

File: src/anymal_c_twins/urdf/leg/haa/haa_3_1_1_macro.urdf.xacro (robot description, xacro)
@@ -13,14 +13,14 @@
     <xacro:property name="min_joint_position"       value="${0.605 + left * 0.115}"/> <!-- [rad] -->
     <!-- joint base HAA -->
-    <joint name="base_${leg}_HAA" type="fixed">
+    <joint name="base_${leg}_HAA_${suffix}" type="fixed">
       <parent link="base_${suffix}"/>
-      <child link="${leg}_HAA"/>
+      <child link="${leg}_HAA_${suffix}"/>
       <origin xyz="${front * B_r_BHaa_x} ${left * B_r_BHaa_y} ${B_r_BHaa_z}"
               rpy="${front*left*q_BHaa_roll} 0 ${(front-1)*0.5*pi}"/>
     </joint>
     <!-- HAA Drive link and joint -->
-    <xacro:include filename="$(find anymal_c)/urdf/leg/drives/drive_${drive_version}_macro.urdf.xacro"/>
-    <xacro:drive name="${leg}_HAA"
-        output="${leg}_HIP"
+    <xacro:include filename="$(find anymal_c_twins)/urdf/leg/drives/drive_${drive_version}_macro.urdf.xacro"/>
+    <xacro:drive name="${leg}_HAA_${suffix}"
+        output="${leg}_HIP_${suffix}"
         direction="${front}"
         enable_collision="${enable_collision}"

File: src/anymal_c_twins/urdf/leg/hfe/hfe_3_1_1_macro.urdf.xacro (robot description, xacro)
@@ -10,13 +10,13 @@
     <xacro:property name="front"        value="${int(leg.startswith('F', 1))*2-1}"/>
     <!-- joint hip HFE -->
-    <joint name="${leg}_hip_fixed_${leg}_HFE" type="fixed">
-      <parent link="${leg}_hip_fixed"/>
-      <child link="${leg}_HFE"/>
+    <joint name="${leg}_hip_fixed_${leg}_HFE_${suffix}" type="fixed">
+      <parent link="${leg}_hip_fixed_${suffix}"/>
+      <child link="${leg}_HFE_${suffix}"/>
       <origin xyz="${front * H_r_HHfe_x} ${left * H_r_HHfe_y} ${H_r_HHfe_z}"
               rpy="0 0 ${left*q_HHfe_yaw}"/>
     </joint>
     <!-- HFE Drive link and joint -->
-    <xacro:include filename="$(find anymal_c)/urdf/leg/drives/drive_${drive_version}_macro.urdf.xacro"/>
-    <xacro:drive name="${leg}_HFE" output="${leg}_THIGH" direction="${left}"/>
+    <xacro:include filename="$(find anymal_c_twins)/urdf/leg/drives/drive_${drive_version}_macro.urdf.xacro"/>
+    <xacro:drive name="${leg}_HFE_${suffix}" output="${leg}_THIGH_${suffix}" direction="${left}"/>
   </xacro:macro>
 </robot>

File: src/anymal_c_twins/urdf/leg/hip/hip_3_1_1_macro.urdf.xacro (robot description, xacro)
@@ -18,16 +18,16 @@
     <xacro:property name="mirrored"     value="${'_mirrored' if left * front == -1 else ''}" />
     <!-- joint HAA hip -->
-    <joint name="${leg}_HIP_${leg}_hip_fixed" type="fixed">
-      <parent link="${leg}_HIP"/>
-      <child link="${leg}_hip_fixed"/>
+    <joint name="${leg}_HIP_${leg}_hip_fixed_${suffix}" type="fixed">
+      <parent link="${leg}_HIP_${suffix}"/>
+      <child link="${leg}_hip_fixed_${suffix}"/>
       <origin xyz="0 0 0" rpy="${left*q_HaaH_roll} 0 ${(front-1)*0.5*pi}"/>
     </joint>
     <!-- Hip link -->
-    <link name="${leg}_hip_fixed">
+    <link name="${leg}_hip_fixed_${suffix}">
      <visual>
        <origin xyz="0 0 0" rpy="0 0 ${(front-1)*0.5*pi}"/>
        <geometry>
          <mesh
-           filename="package://anymal_c/urdf/leg/hip/hip_3_1_1_mesh${mirrored}.dae"
+           filename="package://anymal_c_twins/urdf/leg/hip/hip_3_1_1_mesh${mirrored}.dae"
            scale="${anymal_meshes_scale}"/>
        </geometry>

File: src/anymal_c_twins/urdf/leg/kfe/kfe_3_1_1_macro.urdf.xacro (robot description, xacro)
@@ -10,13 +10,13 @@
     <xacro:property name="front"        value="${int(leg.startswith('F', 1))*2-1}"/>
     <!-- joint thigh KFE -->
-    <joint name="${leg}_thigh_fixed_${leg}_KFE" type="fixed">
-      <parent link="${leg}_thigh_fixed"/>
-      <child link="${leg}_KFE"/>
+    <joint name="${leg}_thigh_fixed_${leg}_KFE_${suffix}" type="fixed">
+      <parent link="${leg}_thigh_fixed_${suffix}"/>
+      <child link="${leg}_KFE_${suffix}"/>
       <origin xyz="${front * T_r_TKfe_x} ${left * T_r_TKfe_y} ${T_r_TKfe_z}"
               rpy="0 0 ${left*q_TKfe_yaw}"/>
     </joint>
     <!-- KFE Drive link and joint -->
-    <xacro:include filename="$(find anymal_c)/urdf/leg/drives/drive_${drive_version}_macro.urdf.xacro"/>
-    <xacro:drive name="${leg}_KFE" output="${leg}_SHANK" direction="${left}"/>
+    <xacro:include filename="$(find anymal_c_twins)/urdf/leg/drives/drive_${drive_version}_macro.urdf.xacro"/>
+    <xacro:drive name="${leg}_KFE_${suffix}" output="${leg}_SHANK_${suffix}" direction="${left}"/>
   </xacro:macro>
 </robot>

File: src/anymal_c_twins/urdf/leg/shank/shank_3_1_1_macro.urdf.xacro (robot description, xacro)
@@ -23,16 +23,16 @@
     <xacro:property name="mirrored"     value="${'_mirrored' if left * front == -1 else ''}" />
     <!-- joint KFE shank -->
-    <joint name="${leg}_shank_${leg}_shank_fixed" type="fixed">
-      <parent link="${leg}_SHANK"/>
-      <child link="${leg}_shank_fixed"/>
+    <joint name="${leg}_shank_${leg}_shank_fixed_${suffix}" type="fixed">
+      <parent link="${leg}_SHANK_${suffix}"/>
+      <child link="${leg}_shank_fixed_${suffix}"/>
       <origin xyz="0 0 0" rpy="0 0 ${left*q_KfeS_yaw}"/>
     </joint>
     <!-- Shank link -->
-    <link name="${leg}_shank_fixed">
+    <link name="${leg}_shank_fixed_${suffix}">
      <visual>
        <origin xyz="0 0 0" rpy="0 0 ${(front-1)*0.5*pi}"/>
        <geometry>
          <mesh
-           filename="package://anymal_c/urdf/leg/shank/shank_3_1_1_mesh${mirrored}.dae"
+           filename="package://anymal_c_twins/urdf/leg/shank/shank_3_1_1_mesh${mirrored}.dae"
            scale="${anymal_meshes_scale}"/>
        </geometry>

File: src/anymal_c_twins/urdf/leg/thigh/thigh_3_1_1_macro.urdf.xacro (robot description, xacro)
@@ -23,16 +23,16 @@
     <xacro:property name="mirrored"     value="${'_mirrored' if left * front == -1 else ''}" />
     <!-- joint HFE thigh -->
-    <joint name="${leg}_THIGH_${leg}_thigh_fixed" type="fixed">
-      <parent link="${leg}_THIGH"/>
-      <child link="${leg}_thigh_fixed"/>
+    <joint name="${leg}_THIGH_${leg}_thigh_fixed_${suffix}" type="fixed">
+      <parent link="${leg}_THIGH_${suffix}"/>
+      <child link="${leg}_thigh_fixed_${suffix}"/>
       <origin xyz="0 0 0" rpy="0 0 ${left*q_HfeT_yaw}"/>
     </joint>
     <!-- Thigh link -->
-    <link name="${leg}_thigh_fixed">
+    <link name="${leg}_thigh_fixed_${suffix}">
       <visual>
         <origin xyz="0 0 0" rpy="0 0 ${(left -1) * 0.5 * pi}"/>
         <geometry>
           <mesh
-               filename="package://anymal_c/urdf/leg/thigh/thigh_3_1_1_mesh.dae"
+               filename="package://anymal_c_twins/urdf/leg/thigh/thigh_3_1_1_mesh.dae"
                scale="${anymal_meshes_scale}"/>
         </geometry>
