Commit message: Successfully load as B. I.e. bugfixes

File: src/anymal_c_twins/urdf/anymal_c_B.urdf.xacro (robot description, xacro)
@@ -45,5 +45,5 @@
   <!-- describes base link (including base intertia dummy link) and integrated sensors-->
   <xacro:if value="${version_ == 'c100'}">
-    <xacro:include filename="$(find anymal_c)/urdf/base/base_3_1_1_macro.urdf.xacro"/>
+    <xacro:include filename="$(find anymal_c_twins)/urdf/base/base_3_1_1_macro.urdf.xacro"/>
     <xacro:base suffix="$(arg suffix)"
                 fix_base="$(arg fix_base)"
@@ -103,14 +103,14 @@
   </xacro:if-->
   <xacro:if value="${version_ == 'c100'}">
-    <xacro:include filename="$(find anymal_c)/urdf/leg/leg_3_1_1_macro.urdf.xacro"/>
+    <xacro:include filename="$(find anymal_c_twins)/urdf/leg/leg_3_1_1_macro.urdf.xacro"/>
   </xacro:if>
-  <xacro:leg leg="LF"/>
-  <xacro:leg leg="RF"/>
-  <xacro:leg leg="LH"/>
-  <xacro:leg leg="RH"/>
+  <xacro:leg leg="LF" suffix="$(arg suffix)"/>
+  <xacro:leg leg="RF" suffix="$(arg suffix)"/>
+  <xacro:leg leg="LH" suffix="$(arg suffix)"/>
+  <xacro:leg leg="RH" suffix="$(arg suffix)"/>
   <!-- Custom payload -->
   <xacro:if value="$(arg enable_custom_payload)">
     <xacro:include filename="$(arg custom_payload_description)"/>
-    <xacro:custom_payload parent="base" />
+    <xacro:custom_payload parent="base_$(arg suffix)" />
   </xacro:if>
   <!-- Inspection payload -->
@@ -118,5 +118,5 @@
   <xacro:if value="$(arg enable_inspection_payload)">
     <xacro:include filename="$(find inspection_payload_description)/urdf/inspection_payload_odrive.urdf.xacro"/>
-    <xacro:inspection_payload name="inspection_payload" parent="base" version="${inspection_payload_version_}">
+    <xacro:inspection_payload name="inspection_payload" parent="base_$(arg suffix)" version="${inspection_payload_version_}">
       <origin xyz="0.116 0.0 0.090" rpy="0 0 0"/>
     </xacro:inspection_payload>
@@ -124,6 +124,6 @@
   <xacro:unless value="$(arg enable_inspection_payload)">
     <!-- describes hatch-->
-    <xacro:include filename="$(find anymal_c)/urdf/base/hatch/hatch_3_1_1_macro.urdf.xacro"/>
-    <xacro:hatch/>
+    <xacro:include filename="$(find anymal_c_twins)/urdf/base/hatch/hatch_3_1_1_macro.urdf.xacro"/>
+    <xacro:hatch suffix="${suffix}"/>
   </xacro:unless>
 </robot>

File: src/anymal_c_twins/urdf/base/base_3_1_1_macro.urdf.xacro (robot description, xacro)
@@ -108,17 +108,17 @@
     <!-- describes shells-->
     <xacro:include filename="$(find anymal_c_twins)/urdf/base/shell/top_shell_3_1_1_macro.urdf.xacro"/>
-    <xacro:top_shell/>
+    <xacro:top_shell suffix="${suffix}"/>
     <xacro:include filename="$(find anymal_c_twins)/urdf/base/shell/bottom_shell_3_1_1_macro.urdf.xacro"/>
-    <xacro:bottom_shell/>
+    <xacro:bottom_shell suffix="${suffix}"/>
     <!-- describes remote-->
     <xacro:include filename="$(find anymal_c_twins)/urdf/base/remote/remote_3_1_1_macro.urdf.xacro"/>
-    <xacro:remote/>
+    <xacro:remote suffix="${suffix}"/>
     <!-- describes handle-->
     <xacro:include filename="$(find anymal_c_twins)/urdf/base/handle/handle_3_1_1_macro.urdf.xacro"/>
-    <xacro:handle/>
+    <xacro:handle suffix="${suffix}"/>
     <!-- describes faces-->
     <xacro:include filename="$(find anymal_c_twins)/urdf/base/face/face_3_1_1_macro.urdf.xacro"/>
-    <xacro:face face="front" simulate_depth_camera="${simulate_depth_camera}" simulate_wide_angle_camera="${simulate_wide_angle_camera}" depth_camera_pitch="${depth_camera_front_pitch}" depth_camera_roll="${depth_camera_front_roll}"/>
-    <xacro:face face="rear"  simulate_depth_camera="${simulate_depth_camera}" simulate_wide_angle_camera="${simulate_wide_angle_camera}" depth_camera_pitch="${depth_camera_rear_pitch}" depth_camera_roll="${depth_camera_rear_roll}"/>
+    <xacro:face suffix="${suffix}" face="front" simulate_depth_camera="${simulate_depth_camera}" simulate_wide_angle_camera="${simulate_wide_angle_camera}" depth_camera_pitch="${depth_camera_front_pitch}" depth_camera_roll="${depth_camera_front_roll}"/>
+    <xacro:face suffix="${suffix}" face="rear"  simulate_depth_camera="${simulate_depth_camera}" simulate_wide_angle_camera="${simulate_wide_angle_camera}" depth_camera_pitch="${depth_camera_rear_pitch}" depth_camera_roll="${depth_camera_rear_roll}"/>
     <!-- describes battery-->
     <xacro:if value="${battery_model == 'travel'}">

File: src/anymal_c_twins/urdf/leg/drives/drive_3_0_2_macro.urdf.xacro (robot description, xacro)
@@ -31,5 +31,5 @@
        <origin xyz="0 0 0" rpy="0 0 0"/>
        <geometry>
-       <mesh filename="package://anymal_c/urdf/leg/drives/drive_3_0_2_mesh.dae"
+       <mesh filename="package://anymal_c_twins/urdf/leg/drives/drive_3_0_2_mesh.dae"
              scale="${anymal_meshes_scale}"/>
        </geometry>

File: src/anymal_c_twins/urdf/leg/leg_3_1_1_macro.urdf.xacro (robot description, xacro)
@@ -3,39 +3,39 @@
   <!-- Leg components -->
   <xacro:macro name="leg" params="leg:=LF suffix:='A' package:=anymal_c_twins">
-    <xacro:haa    leg="${leg}" version="3_1_1" drive_version="3_0_2" package="${package}"/>
-    <xacro:hip    leg="${leg}" version="3_1_1" package="${package}"/>
-    <xacro:hfe    leg="${leg}" version="3_1_1" drive_version="3_0_2" package="${package}"/>
-    <xacro:thigh  leg="${leg}" version="3_1_1" package="${package}"/>
-    <xacro:kfe    leg="${leg}" version="3_1_1" drive_version="3_0_2" package="${package}"/>
-    <xacro:shank  leg="${leg}" version="3_1_1" package="${package}"/>
-    <xacro:foot   leg="${leg}" version="3_1_1" package="${package}"/>
+    <xacro:haa    leg="${leg}" suffix="${suffix}" version="3_1_1" drive_version="3_0_2" package="${package}"/>
+    <xacro:hip    leg="${leg}" suffix="${suffix}" version="3_1_1" package="${package}"/>
+    <xacro:hfe    leg="${leg}" suffix="${suffix}" version="3_1_1" drive_version="3_0_2" package="${package}"/>
+    <xacro:thigh  leg="${leg}" suffix="${suffix}" version="3_1_1" package="${package}"/>
+    <xacro:kfe    leg="${leg}" suffix="${suffix}" version="3_1_1" drive_version="3_0_2" package="${package}"/>
+    <xacro:shank  leg="${leg}" suffix="${suffix}" version="3_1_1" package="${package}"/>
+    <xacro:foot   leg="${leg}" suffix="${suffix}" version="3_1_1" package="${package}"/>
   </xacro:macro>
   <xacro:macro name="haa" params="leg:=LF suffix:='A' version drive_version package">
     <xacro:include filename="$(find ${package})/urdf/leg/haa/haa_${version}_macro.urdf.xacro"/>
-    <xacro:anymal_haa leg="${leg}" drive_version="${drive_version}" enable_collision="false"/>
+    <xacro:anymal_haa leg="${leg}" suffix="${suffix}" drive_version="${drive_version}" enable_collision="false"/>
   </xacro:macro>
   <xacro:macro name="hip" params="leg:=LF suffix:='A' version package">
     <xacro:include filename="$(find ${package})/urdf/leg/hip/hip_${version}_macro.urdf.xacro"/>
-    <xacro:anymal_hip leg="${leg}"/>
+    <xacro:anymal_hip leg="${leg}" suffix="${suffix}"/>
   </xacro:macro>
   <xacro:macro name="hfe" params="leg:=LF suffix:='A' version drive_version package">
     <xacro:include filename="$(find ${package})/urdf/leg/hfe/hfe_${version}_macro.urdf.xacro"/>
-    <xacro:anymal_hfe leg="${leg}" drive_version="${drive_version}"/>
+    <xacro:anymal_hfe leg="${leg}" suffix="${suffix}" drive_version="${drive_version}"/>
   </xacro:macro>
   <xacro:macro name="thigh" params="leg:=LF suffix:='A' version package">
     <xacro:include filename="$(find ${package})/urdf/leg/thigh/thigh_${version}_macro.urdf.xacro"/>
-    <xacro:anymal_thigh leg="${leg}"/>
+    <xacro:anymal_thigh leg="${leg}" suffix="${suffix}"/>
   </xacro:macro>
   <xacro:macro name="kfe" params="leg:=LF suffix:='A' version drive_version package">
     <xacro:include filename="$(find ${package})/urdf/leg/kfe/kfe_${version}_macro.urdf.xacro"/>
-    <xacro:anymal_kfe leg="${leg}" drive_version="${drive_version}"/>
+    <xacro:anymal_kfe leg="${leg}" suffix="${suffix}" drive_version="${drive_version}"/>
   </xacro:macro>
   <xacro:macro name="shank" params="leg:=LF suffix:='A' version package">
     <xacro:include filename="$(find ${package})/urdf/leg/shank/shank_${version}_macro.urdf.xacro"/>
-    <xacro:anymal_shank leg="${leg}"/>
+    <xacro:anymal_shank leg="${leg}" suffix="${suffix}"/>
   </xacro:macro>
   <xacro:macro name="foot" params="leg:=LF suffix:='A' version package">
     <xacro:include filename="$(find ${package})/urdf/leg/foot/foot_${version}_macro.urdf.xacro"/>
-    <xacro:anymal_foot leg="${leg}"/>
+    <xacro:anymal_foot leg="${leg}" suffix="${suffix}"/>
   </xacro:macro>
 </robot>

File: src/anytwin_urdf_development/urdf/anymal_c.urdf.xacro (robot description, xacro)
@@ -4,4 +4,4 @@
         <xacro:include filename="$(find anymal_c_twins)/urdf/anymal_c_${suffix}.urdf.xacro"/>
     </xacro:macro>
-    <xacro:anymal_c_macro suffix='A'/>
+    <xacro:anymal_c_macro suffix='B'/>
 </robot>

File: src/anytwin_urdf_development/urdf/anytwin_c.urdf.xacro (robot description, xacro)
@@ -2,8 +2,13 @@
 <robot name="anymal_c" xmlns:xacro="http://www.ros.org/wiki/xacro">
 <!--include macro to load anymal_c versions A and B-->
-    <xacro:include filename="$(find anytwin_urdf_development)/urdf/anymal_c.urdf.xacro"/>
+    <!--xacro:include filename="$(find anytwin_urdf_development)/urdf/anymal_c.urdf.xacro"/-->
     <xacro:arg name="suffix_one" default="A"/>
     <xacro:arg name="suffix_two" default="B"/>
-    <xacro:anymal_c_macro suffix="$(arg suffix_one)"/>
-    <xacro:anymal_c_macro suffix="$(arg suffix_two)"/>
+    <xacro:macro name="anymal_c_macro" params="suffix">
+        <xacro:include filename="$(find anymal_c_twins)/urdf/anymal_c_${suffix}.urdf.xacro"/>
+    </xacro:macro>
+    <!--xacro:anymal_c_macro suffix="$(arg suffix_one)"/>
+    <xacro:anymal_c_macro suffix="$(arg suffix_two)"/-->
+    <xacro:anymal_c_macro suffix='A'/>
+    <xacro:anymal_c_macro suffix='B'/>
 </robot>
