Commit message: Load anymal A into rviz

File: src/anymal_c_twins/urdf/anymal_c_A.urdf.xacro (robot description, xacro)
@@ -1,5 +1,5 @@
 <?xml version="1.0"?>
 <!-- This file contains the description of the ANYmal robot. -->
-<robot name="anymal" xmlns:xacro="http://www.ros.org/wiki/xacro">
+<robot name="anymal_A" xmlns:xacro="http://www.ros.org/wiki/xacro">
   <!-- Arguments -->
   <xacro:arg name="simulation"                    default="true"/>

File: src/anytwin_urdf_development/urdf/anymal_c.urdf.xacro (robot description, xacro)
@@ -1,7 +1,6 @@
 <?xml version="1.0"?>
 <robot name="anymal_c" xmlns:xacro="http://www.ros.org/wiki/xacro">
-    <xacro:arg name="model" default="$(find anymal_c_renamable)/urdf/anymal_c.urdf.xacro"/>
-    <xacro:macro name="anymal_c_macro">
-        <xacro:include filename="$(find anymal_c)/urdf/anymal_c.urdf.xacro"/>
+    <xacro:macro name="anymal_c_macro" params="suffix:='A'">
+        <xacro:include filename="$(find anymal_c_twins)/urdf/anymal_c_${suffix}.urdf.xacro"/>
     </xacro:macro>
     <xacro:anymal_c_macro/>

Commit message: WIP: crash because of non unique names

File: src/anymal_c_twins/urdf/anymal_c_A.urdf.xacro (robot description, xacro)
@@ -1,5 +1,5 @@
 <?xml version="1.0"?>
 <!-- This file contains the description of the ANYmal robot. -->
-<robot name="anymal_A" xmlns:xacro="http://www.ros.org/wiki/xacro">
+<robot name="anymal_c_A" xmlns:xacro="http://www.ros.org/wiki/xacro">
   <!-- Arguments -->
   <xacro:arg name="simulation"                    default="true"/>

File: src/anymal_c_twins/urdf/anymal_c_B.urdf.xacro (robot description, xacro)
@@ -1,5 +1,5 @@
 <?xml version="1.0"?>
 <!-- This file contains the description of the ANYmal robot. -->
-<robot name="anymal_C" xmlns:xacro="http://www.ros.org/wiki/xacro">
+<robot name="anymal_B" xmlns:xacro="http://www.ros.org/wiki/xacro">
   <!-- Arguments -->
   <xacro:arg name="simulation"                    default="true"/>

File: src/anytwin_urdf_development/urdf/anytwin_c.urdf.xacro (robot description, xacro)
@@ -1,15 +1,9 @@
 <?xml version="1.0"?>
 <robot name="anymal_c" xmlns:xacro="http://www.ros.org/wiki/xacro">
-    <xacro:arg name="model" default="$(find anymal_c_renamable)/urdf/anymal_c_renamable.urdf.xacro"/>
+<!--include macro to load anymal_c versions A and B-->
+    <xacro:include filename="$(find anytwin_urdf_development)/urdf/anymal_c.urdf.xacro"/>
     <xacro:arg name="suffix_one" default="A"/>
-    <cacro:arg name="suffix_two" default="B"/>
-    <xacro:include filename="$(find anymal_c)/urdf/anymal_c.urdf.xacro"/>
-    <xacro:macro name="anymal_c_macro" params="suffix_one_parameter suffix_two_parameter">
-        <!-- one cannot pass arguments (here: suffix_one or suffix_two into included files. I need to make the entire content of anymal_c a macro. Maybe I can then include it and use it here. )-->
-    </xacro:macro>
-    <!--joint name="caster_${suffix}_joint">
-        <axis xyz="0 0 1" />
-    </joint-->
-    <xacro:anymal_c_macro/>
-    <xacro:anymal_c_macro/>
+    <xacro:arg name="suffix_two" default="B"/>
+    <xacro:anymal_c_macro suffix="$(arg suffix_one)"/>
+    <xacro:anymal_c_macro suffix="$(arg suffix_two)"/>
 </robot>

Commit message: WIP: babysteps

File: src/anymal_c_twins/urdf/anymal_c_A.urdf.xacro (robot description, xacro)
@@ -3,5 +3,5 @@
 <robot name="anymal_c_A" xmlns:xacro="http://www.ros.org/wiki/xacro">
   <!-- Arguments -->
-  <xacro:arg name="suffix"                        default="B"/>
+  <xacro:arg name="suffix"                        default="A"/>
   <xacro:arg name="simulation"                    default="true"/>
   <xacro:arg name="perfect_sensors"               default="true"/>
@@ -37,7 +37,7 @@
   <!-- Includes -->
   <!-- describes mesh scale factor and contact model parameters-->
-  <xacro:include filename="$(find anymal_c)/urdf/include/utils.urdf.xacro"/>
+  <xacro:include filename="$(find anymal_c_twins)/urdf/include/utils.urdf.xacro"/>
   <!-- describes gazebo plugin if simulation argument is true-->
-  <xacro:include filename="$(find anymal_c)/urdf/include/plugin.gazebo.xacro"/>
+  <xacro:include filename="$(find anymal_c_twins)/urdf/include/plugin.gazebo.xacro"/>
   <xacro:property name="inspection_payload_version_" value="$(arg inspection_payload_version)"/>
   <xacro:property name="version_" value="$(arg version)"/>
@@ -103,5 +103,5 @@
   </xacro:if-->
   <xacro:if value="${version_ == 'c100'}">
-    <xacro:include filename="$(find anymal_c)/urdf/leg/leg_3_1_1_macro.urdf.xacro"/>
+    <xacro:include filename="$(find anymal_c_twins)/urdf/leg/leg_3_1_1_macro.urdf.xacro"/>
   </xacro:if>
   <xacro:leg leg="LF"/>
@@ -112,5 +112,5 @@
   <xacro:if value="$(arg enable_custom_payload)">
     <xacro:include filename="$(arg custom_payload_description)"/>
-    <xacro:custom_payload parent="base" />
+    <xacro:custom_payload parent="base_$(arg suffix)" />
   </xacro:if>
   <!-- Inspection payload -->
@@ -118,5 +118,5 @@
   <xacro:if value="$(arg enable_inspection_payload)">
     <xacro:include filename="$(find inspection_payload_description)/urdf/inspection_payload_odrive.urdf.xacro"/>
-    <xacro:inspection_payload name="inspection_payload" parent="base" version="${inspection_payload_version_}">
+    <xacro:inspection_payload name="inspection_payload" parent="base_$(arg suffix)" version="${inspection_payload_version_}">
       <origin xyz="0.116 0.0 0.090" rpy="0 0 0"/>
     </xacro:inspection_payload>
@@ -124,5 +124,5 @@
   <xacro:unless value="$(arg enable_inspection_payload)">
     <!-- describes hatch-->
-    <xacro:include filename="$(find anymal_c)/urdf/base/hatch/hatch_3_1_1_macro.urdf.xacro"/>
+    <xacro:include filename="$(find anymal_c_twins)/urdf/base/hatch/hatch_3_1_1_macro.urdf.xacro"/>
     <xacro:hatch/>
   </xacro:unless>

File: src/anymal_c_twins/urdf/anymal_c_B.urdf.xacro (robot description, xacro)
@@ -37,7 +37,7 @@
   <!-- Includes -->
   <!-- describes mesh scale factor and contact model parameters-->
-  <xacro:include filename="$(find anymal_c)/urdf/include/utils.urdf.xacro"/>
+  <xacro:include filename="$(find anymal_c_twins)/urdf/include/utils.urdf.xacro"/>
   <!-- describes gazebo plugin if simulation argument is true-->
-  <xacro:include filename="$(find anymal_c)/urdf/include/plugin.gazebo.xacro"/>
+  <xacro:include filename="$(find anymal_c_twins)/urdf/include/plugin.gazebo.xacro"/>
   <xacro:property name="inspection_payload_version_" value="$(arg inspection_payload_version)"/>
   <xacro:property name="version_" value="$(arg version)"/>

File: src/anymal_c_twins/urdf/base/base_3_1_1_macro.urdf.xacro (robot description, xacro)
@@ -1,5 +1,6 @@
 <?xml version="1.0"?>
 <robot xmlns:xacro="http://www.ros.org/wiki/xacro">
-  <xacro:macro name="base" params="fix_base:=false
+  <xacro:macro name="base" params="suffix:='A'
+                                   fix_base:=false
                                    simulate_depth_camera:=false
                                    simulate_lidar:=false
@@ -36,5 +37,5 @@
       <gazebo>
         <joint name="world_joint" type="fixed">
-          <parent>base</parent>
+          <parent>base_${suffix}</parent>
           <child>world</child>
         </joint>
@@ -42,10 +43,10 @@
     </xacro:if>
     <!-- Base link -->
-    <link name="base">
+    <link name="base_${suffix}">
       <visual>
         <origin xyz="0 0 0" rpy="0 0 0"/>
         <geometry>
           <mesh
-            filename="package://anymal_c/urdf/base/base_3_1_1_mesh.dae"
+            filename="package://anymal_c_twins/urdf/base/base_3_1_1_mesh.dae"
             scale="${anymal_meshes_scale}"/>
         </geometry>
@@ -90,11 +91,11 @@
     </link>
     <!-- Fixed joint to add dummy inertia link -->
-    <joint name="base_to_base_inertia" type="fixed">
-      <parent link="base"/>
-      <child link="base_inertia"/>
+    <joint name="base_to_base_inertia_${suffix}" type="fixed">
+      <parent link="base_${suffix}"/>
+      <child link="base_inertia_${suffix}"/>
       <origin xyz="0 0 0" rpy="0 0 0"/>
     </joint>
     <!-- Dummy inertia link, because KDL cannot have inertia on the base link -->
-    <link name="base_inertia">
+    <link name="base_inertia_${suffix}">
       <inertial>
         <origin   xyz="${B_r_BBcom_x} ${B_r_BBcom_y} ${B_r_BBcom_z}"
@@ -106,52 +107,52 @@
     </link>
     <!-- describes shells-->
-    <xacro:include filename="$(find anymal_c)/urdf/base/shell/top_shell_3_1_1_macro.urdf.xacro"/>
+    <xacro:include filename="$(find anymal_c_twins)/urdf/base/shell/top_shell_3_1_1_macro.urdf.xacro"/>
     <xacro:top_shell/>
-    <xacro:include filename="$(find anymal_c)/urdf/base/shell/bottom_shell_3_1_1_macro.urdf.xacro"/>
+    <xacro:include filename="$(find anymal_c_twins)/urdf/base/shell/bottom_shell_3_1_1_macro.urdf.xacro"/>
     <xacro:bottom_shell/>
     <!-- describes remote-->
-    <xacro:include filename="$(find anymal_c)/urdf/base/remote/remote_3_1_1_macro.urdf.xacro"/>
+    <xacro:include filename="$(find anymal_c_twins)/urdf/base/remote/remote_3_1_1_macro.urdf.xacro"/>
     <xacro:remote/>
     <!-- describes handle-->
-    <xacro:include filename="$(find anymal_c)/urdf/base/handle/handle_3_1_1_macro.urdf.xacro"/>
+    <xacro:include filename="$(find anymal_c_twins)/urdf/base/handle/handle_3_1_1_macro.urdf.xacro"/>
     <xacro:handle/>
     <!-- describes faces-->
-    <xacro:include filename="$(find anymal_c)/urdf/base/face/face_3_1_1_macro.urdf.xacro"/>
+    <xacro:include filename="$(find anymal_c_twins)/urdf/base/face/face_3_1_1_macro.urdf.xacro"/>
     <xacro:face face="front" simulate_depth_camera="${simulate_depth_camera}" simulate_wide_angle_camera="${simulate_wide_angle_camera}" depth_camera_pitch="${depth_camera_front_pitch}" depth_camera_roll="${depth_camera_front_roll}"/>
     <xacro:face face="rear"  simulate_depth_camera="${simulate_depth_camera}" simulate_wide_angle_camera="${simulate_wide_angle_camera}" depth_camera_pitch="${depth_camera_rear_pitch}" depth_camera_roll="${depth_camera_rear_roll}"/>
     <!-- describes battery-->
     <xacro:if value="${battery_model == 'travel'}">
-      <xacro:include filename="$(find anymal_c)/urdf/base/battery/travel_battery_3_0_5_macro.urdf.xacro"/>
+      <xacro:include filename="$(find anymal_c_twins)/urdf/base/battery/travel_battery_3_0_5_macro.urdf.xacro"/>
     </xacro:if>
     <xacro:if value="${battery_model == 'regular'}">
-      <xacro:include filename="$(find anymal_c)/urdf/base/battery/battery_3_0_4_macro.urdf.xacro"/>
+      <xacro:include filename="$(find anymal_c_twins)/urdf/base/battery/battery_3_0_4_macro.urdf.xacro"/>
     </xacro:if>
     <xacro:battery/>
     <!-- describes docking socket/hatch-->
     <xacro:if value="${docking_socket}">
-      <xacro:include filename="$(find anymal_c)/urdf/base/docking_hatch/docking_socket_3_1_1_macro.urdf.xacro"/>
+      <xacro:include filename="$(find anymal_c_twins)/urdf/base/docking_hatch/docking_socket_3_1_1_macro.urdf.xacro"/>
       <xacro:docking_socket/>
     </xacro:if>
     <xacro:unless value="${docking_socket}">
-      <xacro:include filename="$(find anymal_c)/urdf/base/docking_hatch/docking_hatch_cover_3_1_1_macro.urdf.xacro"/>
+      <xacro:include filename="$(find anymal_c_twins)/urdf/base/docking_hatch/docking_hatch_cover_3_1_1_macro.urdf.xacro"/>
       <xacro:docking_hatch_cover/>
     </xacro:unless>
     <!-- Epson IMU -->
     <xacro:include filename="$(find any_description)/urdf/sensors/imu/epson/epson.urdf.xacro"/>
-    <xacro:epson name="imu" parent="base" update_rate="400" ns="sensors" frame_id="imu_link" topic_name="imu">
+    <xacro:epson name="imu" parent="base_${suffix}" update_rate="400" ns="sensors" frame_id="imu_link" topic_name="imu">
         <origin xyz="0.2488 0.00835 0.04628" rpy="${imu_roll/180*pi} ${imu_pitch/180*pi} ${imu_yaw/180*pi}"/>
     </xacro:epson>
     <!-- Realsense left -->
-    <xacro:include filename="$(find anymal_c)/urdf/base/sensors/depth_camera/realsense_d435_3_1_1.urdf.xacro"/>
-    <xacro:anymal_realsense name="depth_camera_left" parent="base" simulation="${simulate_depth_camera}">
+    <xacro:include filename="$(find anymal_c_twins)/urdf/base/sensors/depth_camera/realsense_d435_3_1_1.urdf.xacro"/>
+    <xacro:anymal_realsense name="depth_camera_left" parent="base_${suffix}" simulation="${simulate_depth_camera}">
       <origin xyz="0.0 0.07646 0.02905" rpy="${depth_camera_left_roll/180*pi} ${depth_camera_left_pitch/180*pi} ${pi/2}"/>
     </xacro:anymal_realsense>
     <!-- Realsense right -->
-    <xacro:anymal_realsense name="depth_camera_right" parent="base" simulation="${simulate_depth_camera}">
+    <xacro:anymal_realsense name="depth_camera_right" parent="base_${suffix}" simulation="${simulate_depth_camera}">
       <origin xyz="0.0 -0.07646 0.02905" rpy="${depth_camera_right_roll/180*pi} ${depth_camera_right_pitch/180*pi} ${-pi/2}"/>
     </xacro:anymal_realsense>
     <!-- Velodyne -->
-    <xacro:include filename="$(find anymal_c)/urdf/base/sensors/lidar/velodyne_3_1_1.urdf.xacro"/>
-    <xacro:anymal_velodyne name="lidar" parent="base" simulation="${simulate_lidar}" yaw="${-pi/2}">
+    <xacro:include filename="$(find anymal_c_twins)/urdf/base/sensors/lidar/velodyne_3_1_1.urdf.xacro"/>
+    <xacro:anymal_velodyne name="lidar" parent="base_${suffix}" simulation="${simulate_lidar}" yaw="${-pi/2}">
       <origin xyz="-0.364 0.0 0.0735" rpy="0 0 0"/>
     </xacro:anymal_velodyne>

File: src/anymal_c_twins/urdf/leg/haa/haa_3_1_1_macro.urdf.xacro (robot description, xacro)
@@ -1,5 +1,5 @@
 <?xml version="1.0"?>
 <robot xmlns:xacro="http://www.ros.org/wiki/xacro">
-  <xacro:macro name="anymal_haa" params="leg:=LF drive_version enable_collision:=true">
+  <xacro:macro name="anymal_haa" params="leg:=LF suffix:='A' drive_version enable_collision:=true">
     <xacro:property name="B_r_BHaa_x"   value= "0.2999"/><!-- [m] -->
     <xacro:property name="B_r_BHaa_y"   value= "0.104"/><!-- [m] -->
@@ -14,5 +14,5 @@
     <!-- joint base HAA -->
     <joint name="base_${leg}_HAA" type="fixed">
-      <parent link="base"/>
+      <parent link="base_${suffix}"/>
       <child link="${leg}_HAA"/>
       <origin xyz="${front * B_r_BHaa_x} ${left * B_r_BHaa_y} ${B_r_BHaa_z}"

File: src/anymal_c_twins/urdf/leg/hfe/hfe_3_1_1_macro.urdf.xacro (robot description, xacro)
@@ -1,5 +1,5 @@
 <?xml version="1.0"?>
 <robot xmlns:xacro="http://www.ros.org/wiki/xacro">
-  <xacro:macro name="anymal_hfe" params="leg:=LF drive_version">
+  <xacro:macro name="anymal_hfe" params="leg:=LF suffix:='A' drive_version">
     <xacro:property name="H_r_HHfe_x"   value= "0.0599"/><!-- [m] -->
     <xacro:property name="H_r_HHfe_y"   value= "0.08381"/><!-- [m] -->

File: src/anymal_c_twins/urdf/leg/hip/hip_3_1_1_macro.urdf.xacro (robot description, xacro)
@@ -1,5 +1,5 @@
 <?xml version="1.0"?>
 <robot xmlns:xacro="http://www.ros.org/wiki/xacro">
-  <xacro:macro name="anymal_hip" params="leg:=LF">
+  <xacro:macro name="anymal_hip" params="leg:=LF suffix:='A'">
     <xacro:property name="q_HaaH_roll"  value= "${-150/180*pi}"/> <!-- [rad] -->
     <xacro:property name="H_r_HHcom_x"  value= "0.048"/> <!-- [m] -->

File: src/anymal_c_twins/urdf/leg/kfe/kfe_3_1_1_macro.urdf.xacro (robot description, xacro)
@@ -1,5 +1,5 @@
 <?xml version="1.0"?>
 <robot xmlns:xacro="http://www.ros.org/wiki/xacro">
-  <xacro:macro name="anymal_kfe" params="leg:=LF drive_version">
+  <xacro:macro name="anymal_kfe" params="leg:=LF suffix:='A' drive_version">
     <xacro:property name="T_r_TKfe_x"   value="0.0"/><!-- [m] -->
     <xacro:property name="T_r_TKfe_y"   value="0.1003"/><!-- [m] -->

File: src/anymal_c_twins/urdf/leg/leg_3_1_1_macro.urdf.xacro (robot description, xacro)
@@ -2,5 +2,5 @@
 <robot name="anymal" xmlns:xacro="http://www.ros.org/wiki/xacro">
   <!-- Leg components -->
-  <xacro:macro name="leg" params="leg:=LF package:=anymal_c">
+  <xacro:macro name="leg" params="leg:=LF suffix:='A' package:=anymal_c_twins">
     <xacro:haa    leg="${leg}" version="3_1_1" drive_version="3_0_2" package="${package}"/>
     <xacro:hip    leg="${leg}" version="3_1_1" package="${package}"/>
@@ -11,29 +11,29 @@
     <xacro:foot   leg="${leg}" version="3_1_1" package="${package}"/>
   </xacro:macro>
-  <xacro:macro name="haa" params="leg:=LF version drive_version package">
+  <xacro:macro name="haa" params="leg:=LF suffix:='A' version drive_version package">
     <xacro:include filename="$(find ${package})/urdf/leg/haa/haa_${version}_macro.urdf.xacro"/>
     <xacro:anymal_haa leg="${leg}" drive_version="${drive_version}" enable_collision="false"/>
   </xacro:macro>
-  <xacro:macro name="hip" params="leg:=LF version package">
+  <xacro:macro name="hip" params="leg:=LF suffix:='A' version package">
     <xacro:include filename="$(find ${package})/urdf/leg/hip/hip_${version}_macro.urdf.xacro"/>
     <xacro:anymal_hip leg="${leg}"/>
   </xacro:macro>
-  <xacro:macro name="hfe" params="leg:=LF version drive_version package">
+  <xacro:macro name="hfe" params="leg:=LF suffix:='A' version drive_version package">
     <xacro:include filename="$(find ${package})/urdf/leg/hfe/hfe_${version}_macro.urdf.xacro"/>
     <xacro:anymal_hfe leg="${leg}" drive_version="${drive_version}"/>
   </xacro:macro>
-  <xacro:macro name="thigh" params="leg:=LF version package">
+  <xacro:macro name="thigh" params="leg:=LF suffix:='A' version package">
     <xacro:include filename="$(find ${package})/urdf/leg/thigh/thigh_${version}_macro.urdf.xacro"/>
     <xacro:anymal_thigh leg="${leg}"/>
   </xacro:macro>
-  <xacro:macro name="kfe" params="leg:=LF version drive_version package">
+  <xacro:macro name="kfe" params="leg:=LF suffix:='A' version drive_version package">
     <xacro:include filename="$(find ${package})/urdf/leg/kfe/kfe_${version}_macro.urdf.xacro"/>
     <xacro:anymal_kfe leg="${leg}" drive_version="${drive_version}"/>
   </xacro:macro>
-  <xacro:macro name="shank" params="leg:=LF version package">
+  <xacro:macro name="shank" params="leg:=LF suffix:='A' version package">
     <xacro:include filename="$(find ${package})/urdf/leg/shank/shank_${version}_macro.urdf.xacro"/>
     <xacro:anymal_shank leg="${leg}"/>
   </xacro:macro>
-  <xacro:macro name="foot" params="leg:=LF version package">
+  <xacro:macro name="foot" params="leg:=LF suffix:='A' version package">
     <xacro:include filename="$(find ${package})/urdf/leg/foot/foot_${version}_macro.urdf.xacro"/>
     <xacro:anymal_foot leg="${leg}"/>

File: src/anymal_c_twins/urdf/leg/shank/shank_3_1_1_macro.urdf.xacro (robot description, xacro)
@@ -1,5 +1,5 @@
 <?xml version="1.0"?>
 <robot xmlns:xacro="http://www.ros.org/wiki/xacro">
-  <xacro:macro name="anymal_shank" params="leg:=LF">
+  <xacro:macro name="anymal_shank" params="leg:=LF suffix:='A'">
     <xacro:property name="q_KfeS_yaw"             value="${-0.5*pi}"/> <!-- [rad] -->
     <xacro:property name="S_r_SScom_x"            value="0.03463"/> <!-- [m] -->

File: src/anymal_c_twins/urdf/leg/thigh/thigh_3_1_1_macro.urdf.xacro (robot description, xacro)
@@ -1,5 +1,5 @@
 <?xml version="1.0"?>
 <robot xmlns:xacro="http://www.ros.org/wiki/xacro">
-  <xacro:macro name="anymal_thigh" params="leg:=LF">
+  <xacro:macro name="anymal_thigh" params="leg:=LF suffix:='A'">
     <xacro:property name="q_HfeT_yaw"       value="${-0.5*pi}"/> <!-- [rad] -->
     <xacro:property name="T_r_TTcom_x"      value="0.0"/> <!-- [m] -->

File: src/anytwin_urdf_development/urdf/anymal_c.urdf.xacro (robot description, xacro)
@@ -4,4 +4,4 @@
         <xacro:include filename="$(find anymal_c_twins)/urdf/anymal_c_${suffix}.urdf.xacro"/>
     </xacro:macro>
-    <xacro:anymal_c_macro/>
+    <xacro:anymal_c_macro suffix='A'/>
 </robot>
