Commit message: Step

File: src/anymal_c_twins/urdf/anymal_c_A.urdf.xacro (robot description, xacro)
@@ -105,8 +105,8 @@
     <xacro:include filename="$(find anymal_c_twins)/urdf/leg/leg_3_1_1_macro.urdf.xacro"/>
   </xacro:if>
-  <xacro:leg leg="LF"/>
-  <xacro:leg leg="RF"/>
-  <xacro:leg leg="LH"/>
-  <xacro:leg leg="RH"/>
+  <xacro:leg leg="LF" suffix="$(arg suffix)"/>
+  <xacro:leg leg="RF" suffix="$(arg suffix)"/>
+  <xacro:leg leg="LH" suffix="$(arg suffix)"/>
+  <xacro:leg leg="RH" suffix="$(arg suffix)"/>
   <!-- Custom payload -->
   <xacro:if value="$(arg enable_custom_payload)">

File: src/anymal_c_twins/urdf/base/base_3_1_1_macro.urdf.xacro (robot description, xacro)
@@ -36,5 +36,5 @@
     <xacro:if value="${fix_base}">
       <gazebo>
-        <joint name="world_joint" type="fixed">
+        <joint name="world_joint_${suffix}" type="fixed">
           <parent>base_${suffix}</parent>
           <child>world</child>
@@ -128,13 +128,13 @@
       <xacro:include filename="$(find anymal_c_twins)/urdf/base/battery/battery_3_0_4_macro.urdf.xacro"/>
     </xacro:if>
-    <xacro:battery/>
+    <xacro:battery suffix="${suffix}"/>
     <!-- describes docking socket/hatch-->
     <xacro:if value="${docking_socket}">
       <xacro:include filename="$(find anymal_c_twins)/urdf/base/docking_hatch/docking_socket_3_1_1_macro.urdf.xacro"/>
-      <xacro:docking_socket/>
+      <xacro:docking_socket suffix="${suffix}"/>
     </xacro:if>
     <xacro:unless value="${docking_socket}">
       <xacro:include filename="$(find anymal_c_twins)/urdf/base/docking_hatch/docking_hatch_cover_3_1_1_macro.urdf.xacro"/>
-      <xacro:docking_hatch_cover/>
+      <xacro:docking_hatch_cover suffix="${suffix}"/>
     </xacro:unless>
     <!-- Epson IMU -->

File: src/anymal_c_twins/urdf/base/battery/battery_3_0_4_macro.urdf.xacro (robot description, xacro)
@@ -1,5 +1,5 @@
 <?xml version="1.0"?>
 <robot xmlns:xacro="http://www.ros.org/wiki/xacro">
-  <xacro:macro name="battery">
+  <xacro:macro name="battery" params="suffix:='A'">
     <xacro:property name="B_r_BBbcom_x" value="-0.00067"/> <!--  [m] -->
     <xacro:property name="B_r_BBbcom_y" value="-0.00023"/> <!--  [m] -->
@@ -13,16 +13,16 @@
     <xacro:property name="B_Iyz_Bb"     value= "0.00000142902"/> <!-- [kg * m^2] -->
     <!-- Fixed joint base battery -->
-    <joint name="base_battery" type="fixed">
-      <parent link="base"/>
-      <child link="battery"/>
+    <joint name="base_battery_${suffix}" type="fixed">
+      <parent link="base_${suffix}"/>
+      <child link="battery_${suffix}"/>
       <origin xyz="0 0 0" rpy="0 0 0"/>
     </joint>
     <!-- Shell link -->
-    <link name="battery">
+    <link name="battery_${suffix}">
       <visual>
         <origin xyz="0 0 0" rpy="0 0 0"/>
        <geometry>
           <mesh
-            filename="package://anymal_c/urdf/base/battery/battery_3_0_4_mesh.dae"
+            filename="package://anymal_c_twins/urdf/base/battery/battery_3_0_4_mesh.dae"
             scale="${anymal_meshes_scale}"/>
         </geometry>

File: src/anymal_c_twins/urdf/base/docking_hatch/docking_hatch_cover_3_1_1_macro.urdf.xacro (robot description, xacro)
@@ -1,5 +1,5 @@
 <?xml version="1.0"?>
 <robot xmlns:xacro="http://www.ros.org/wiki/xacro">
-  <xacro:macro name="docking_hatch_cover">
+  <xacro:macro name="docking_hatch_cover" params="suffix:='A'">
     <xacro:property name="Dhc_r_Dhccom_x"  value= "-0.003"/> <!--  [m] -->
     <xacro:property name="Dhc_r_Dhccom_y"  value= "0.0"/> <!--  [m] -->
@@ -13,11 +13,11 @@
     <xacro:property name="Dhc_Iyz_Dhc"     value= "0.0"/> <!-- [kg * m^2] -->
     <!-- Fixed joint to add docking  -->
-    <joint name="base_to_docking_hatch_cover" type="fixed">
-      <parent link="base"/>
-      <child link="docking_hatch_cover"/>
+    <joint name="base_to_docking_hatch_cover_${suffix}" type="fixed">
+      <parent link="base_${suffix}"/>
+      <child link="docking_hatch_cover_${suffix}"/>
       <origin xyz="0.343 0.0 -0.07" rpy="0 0 0"/>
     </joint>
     <!-- Hatch cover link -->
-    <link name="docking_hatch_cover">
+    <link name="docking_hatch_cover_${suffix}">
       <!--  TODO(fgiraldez): add visual    -->
       <inertial>

File: src/anymal_c_twins/urdf/base/docking_hatch/docking_socket_3_1_1_macro.urdf.xacro (robot description, xacro)
@@ -1,5 +1,5 @@
 <?xml version="1.0"?>
 <robot xmlns:xacro="http://www.ros.org/wiki/xacro">
-  <xacro:macro name="docking_socket">
+  <xacro:macro name="docking_socket" params="suffix:='A'">
     <xacro:property name="Ds_r_Dscom_x"  value= "-0.002"/> <!--  [m] -->
     <xacro:property name="Ds_r_Dscom_y"  value= "-0.001"/> <!--  [m] -->
@@ -13,11 +13,11 @@
     <xacro:property name="Ds_Iyz_Ds"     value= "0.000002760"/> <!-- [kg * m^2] -->
     <!-- Fixed joint to add docking  -->
-    <joint name="base_to_docking_socket" type="fixed">
-      <parent link="base"/>
-      <child link="docking_socket"/>
+    <joint name="base_to_docking_socket_${suffix}" type="fixed">
+      <parent link="base_${suffix}"/>
+      <child link="docking_socket_${suffix}"/>
       <origin xyz="0.343 0.0 -0.07" rpy="0 0 0"/>
     </joint>
     <!-- Hatch cover link -->
-    <link name="docking_socket">
+    <link name="docking_socket_${suffix}">
       <!--  TODO(fgiraldez): add visual    -->
       <inertial>

File: src/anymal_c_twins/urdf/base/face/face_3_1_1_macro.urdf.xacro (robot description, xacro)
@@ -1,5 +1,5 @@
 <?xml version="1.0"?>
 <robot xmlns:xacro="http://www.ros.org/wiki/xacro">
-  <xacro:macro name="face" params="face simulate_depth_camera:=false simulate_wide_angle_camera:=false depth_camera_pitch:=30 depth_camera_roll:=0">
+  <xacro:macro name="face" params="suffix:='A' face simulate_depth_camera:=false simulate_wide_angle_camera:=false depth_camera_pitch:=30 depth_camera_roll:=0">
     <xacro:property name="B_r_BBf_x"        value="0.41450"/> <!--  [m] -->
     <xacro:property name="B_r_BBf_z"        value="0.00700"/> <!--  [m] -->
@@ -20,16 +20,16 @@
     <xacro:property name="direction"    value="${1 if face == 'front' else -1}"/>
     <!-- Fixed joint base face -->
-    <joint name="base_face_${face}" type="fixed">
-      <parent link="base"/>
-      <child link="face_${face}"/>
+    <joint name="base_face_${face}_${suffix}" type="fixed">
+      <parent link="base_${suffix}"/>
+      <child link="face_${face}_${suffix}"/>
       <origin xyz="${direction * B_r_BBf_x} 0 0" rpy="0 0 ${-0.5*(direction-1) * pi}"/>
     </joint>
     <!-- Shell link -->
-    <link name="face_${face}">
+    <link name="face_${face}_${suffix}">
       <visual>
         <origin xyz="0 0 0" rpy="0 0 0"/>
        <geometry>
           <mesh
-            filename="package://anymal_c/urdf/base/face/face_3_1_1_mesh.dae"
+            filename="package://anymal_c_twins/urdf/base/face/face_3_1_1_mesh.dae"
             scale="1.0 1.0 1.0"/>
        </geometry>
@@ -62,11 +62,11 @@
     </link>
     <!-- Depth Camera -->
-    <xacro:include filename="$(find anymal_c)/urdf/base/sensors/depth_camera/realsense_d435_3_1_1.urdf.xacro"/>
-    <xacro:anymal_realsense name="depth_camera_${face}" parent="face_${face}" simulation="${simulate_depth_camera}">
+    <xacro:include filename="$(find anymal_c_twins)/urdf/base/sensors/depth_camera/realsense_d435_3_1_1.urdf.xacro"/>
+    <xacro:anymal_realsense name="depth_camera_${face}_${suffix}" parent="face_${face}_${suffix}" simulation="${simulate_depth_camera}">
       <origin xyz="0.04715 0.0 -0.0292" rpy="${depth_camera_roll/180*pi} ${depth_camera_pitch/180*pi} 0"/>
     </xacro:anymal_realsense>
     <!-- Wide Angle Camera -->
-    <xacro:include filename="$(find anymal_c)/urdf/base/sensors/wide_angle_camera/blackfly_s_3_1_1.urdf.xacro"/>
-    <xacro:blackfly name="wide_angle_camera_${face}" parent="face_${face}" simulation="${simulate_wide_angle_camera}" fps="30.0">
+    <xacro:include filename="$(find anymal_c_twins)/urdf/base/sensors/wide_angle_camera/blackfly_s_3_1_1.urdf.xacro"/>
+    <xacro:blackfly name="wide_angle_camera_${face}_${suffix}" parent="face_${face}_${suffix}" simulation="${simulate_wide_angle_camera}" fps="30.0">
       <origin xyz="0.09850 0.0 0.01497" rpy="0 0 0"/>
     </xacro:blackfly>

File: src/anymal_c_twins/urdf/base/handle/handle_3_1_1_macro.urdf.xacro (robot description, xacro)
@@ -1,5 +1,5 @@
 <?xml version="1.0"?>
 <robot xmlns:xacro="http://www.ros.org/wiki/xacro">
-  <xacro:macro name="handle">
+  <xacro:macro name="handle" params="suffix:='A'">
     <xacro:property name="B_r_BBbcom_x" value= "0.37801"/> <!--  [m] -->
     <xacro:property name="B_r_BBbcom_y" value= "0.0"/> <!--  [m] -->
@@ -13,16 +13,16 @@
     <xacro:property name="B_Iyz_Bb"     value= "0.000000001"/> <!-- [kg * m^2] -->
     <!-- Fixed joint base handle -->
-    <joint name="base_handle" type="fixed">
-      <parent link="base"/>
-      <child link="handle"/>
+    <joint name="base_handle_${suffix}" type="fixed">
+      <parent link="base_${suffix}"/>
+      <child link="handle_${suffix}"/>
       <origin xyz="0 0 0" rpy="0 0 0"/>
     </joint>
     <!-- Handle link -->
-    <link name="handle">
+    <link name="handle_${suffix}">
       <visual>
         <origin xyz="0 0 0" rpy="0 0 0"/>
         <geometry>
           <mesh
-            filename="package://anymal_c/urdf/base/handle/handle_3_1_1_mesh.dae"
+            filename="package://anymal_c_twins/urdf/base/handle/handle_3_1_1_mesh.dae"
             scale="${anymal_meshes_scale}"/>
         </geometry>

File: src/anymal_c_twins/urdf/base/hatch/hatch_3_1_1_macro.urdf.xacro (robot description, xacro)
@@ -1,5 +1,5 @@
 <?xml version="1.0"?>
 <robot xmlns:xacro="http://www.ros.org/wiki/xacro">
-  <xacro:macro name="hatch">
+  <xacro:macro name="hatch" params="suffix:='A'">
     <xacro:property name="B_r_BBh_x"      value= "0.0"/> <!--  [m] -->
     <xacro:property name="B_r_BBh_y"      value= "0.0"/> <!--  [m] -->
@@ -16,15 +16,15 @@
     <xacro:property name="Bh_Iyz_Bh"      value= "0.001"/> <!-- [kg * m^2] -->
     <!-- Fixed joint base hatch -->
-    <joint name="base_hatch" type="fixed">
-      <parent link="base"/>
-      <child link="hatch"/>
+    <joint name="base_hatch_${suffix}" type="fixed">
+      <parent link="base_${suffix}"/>
+      <child link="hatch_${suffix}"/>
       <origin xyz="${B_r_BBh_x} ${B_r_BBh_y} ${B_r_BBh_z}" rpy="0 0 0"/>
     </joint>
     <!-- Hatch link -->
-    <link name="hatch">
+    <link name="hatch_${suffix}">
       <visual>
         <origin xyz="0.116 0 0.073" rpy="0 0 0"/>
         <geometry>
-          <mesh filename="package://anymal_c/urdf/base/hatch/hatch_3_1_1_mesh.dae"
+          <mesh filename="package://anymal_c_twins/urdf/base/hatch/hatch_3_1_1_mesh.dae"
                 scale="1.0 1.0 1.0"/>
         </geometry>

File: src/anymal_c_twins/urdf/base/remote/remote_3_1_1_macro.urdf.xacro (robot description, xacro)
@@ -1,5 +1,5 @@
 <?xml version="1.0"?>
 <robot xmlns:xacro="http://www.ros.org/wiki/xacro">
-  <xacro:macro name="remote">
+  <xacro:macro name="remote" params="suffix:='A'">
     <xacro:property name="B_r_BBbcom_x" value="-0.171"/> <!--  [m] -->
     <xacro:property name="B_r_BBbcom_y" value= "0.002"/> <!--  [m] -->
@@ -13,16 +13,16 @@
     <xacro:property name="B_Iyz_Bb"     value= "0.000000740"/> <!-- [kg * m^2] -->
     <!-- Fixed joint base remote -->
-    <joint name="base_remote" type="fixed">
-      <parent link="base"/>
-      <child link="remote"/>
+    <joint name="base_remote_${suffix}" type="fixed">
+      <parent link="base_${suffix}"/>
+      <child link="remote_${suffix}"/>
       <origin xyz="0 0 0" rpy="0 0 0"/>
     </joint>
     <!-- Remote link -->
-    <link name="remote">
+    <link name="remote_${suffix}">
       <visual>
         <origin xyz="0 0 0" rpy="0 0 0"/>
        <geometry>
           <mesh
-            filename="package://anymal_c/urdf/base/remote/remote_3_1_1_mesh.dae"
+            filename="package://anymal_c_twins/urdf/base/remote/remote_3_1_1_mesh.dae"
             scale="${anymal_meshes_scale}"/>
         </geometry>

File: src/anymal_c_twins/urdf/base/shell/bottom_shell_3_1_1_macro.urdf.xacro (robot description, xacro)
@@ -1,5 +1,5 @@
 <?xml version="1.0"?>
 <robot xmlns:xacro="http://www.ros.org/wiki/xacro">
-  <xacro:macro name="bottom_shell">
+  <xacro:macro name="bottom_shell" params="suffix:='A'">
     <xacro:property name="B_r_BBscom_x"        value="-0.00333"/> <!--  [m] -->
     <xacro:property name="B_r_BBscom_y"        value= "0.00001"/> <!--  [m] -->
@@ -14,5 +14,5 @@
     <!-- Fixed joint base topshell -->
     <joint name="base_bottom_shell" type="fixed">
-      <parent link="base"/>
+      <parent link="base_${suffix}"/>
       <child link="bottom_shell"/>
       <origin xyz="0 0 0" rpy="0 0 0"/>
@@ -24,5 +24,5 @@
         <geometry>
           <mesh
-            filename="package://anymal_c/urdf/base/shell/bottom_shell_3_1_1_mesh.dae"
+            filename="package://anymal_c_twins/urdf/base/shell/bottom_shell_3_1_1_mesh.dae"
             scale="1.0 1.0 1.0"/>
         </geometry>

File: src/anymal_c_twins/urdf/base/shell/top_shell_3_1_1_macro.urdf.xacro (robot description, xacro)
@@ -1,5 +1,5 @@
 <?xml version="1.0"?>
 <robot xmlns:xacro="http://www.ros.org/wiki/xacro">
-  <xacro:macro name="top_shell">
+  <xacro:macro name="top_shell" params="suffix:='A'">
     <xacro:property name="B_r_BBscom_x"        value="-0.00777"/> <!--  [m] -->
     <xacro:property name="B_r_BBscom_y"        value="-0.00013"/> <!--  [m] -->
@@ -14,5 +14,5 @@
     <!-- Fixed joint base topshell -->
     <joint name="base_top_shell" type="fixed">
-      <parent link="base"/>
+      <parent link="base_${suffix}"/>
       <child link="top_shell"/>
       <origin xyz="0 0 0" rpy="0 0 0"/>
@@ -24,5 +24,5 @@
         <geometry>
           <mesh
-            filename="package://anymal_c/urdf/base/shell/top_shell_3_1_1_mesh.dae"
+            filename="package://anymal_c_twins/urdf/base/shell/top_shell_3_1_1_mesh.dae"
             scale="1.0 1.0 1.0"/>
         </geometry>

Commit message: AnyTwin load from xacro working

File: src/anymal_c_twins/urdf/anymal_c_A.urdf.xacro (robot description, xacro)
@@ -125,5 +125,5 @@
     <!-- describes hatch-->
     <xacro:include filename="$(find anymal_c_twins)/urdf/base/hatch/hatch_3_1_1_macro.urdf.xacro"/>
-    <xacro:hatch/>
+    <xacro:hatch suffix="${suffix}"/>
   </xacro:unless>
 </robot>

File: src/anymal_c_twins/urdf/anymal_c_B.urdf.xacro (robot description, xacro)
@@ -3,5 +3,5 @@
 <robot name="anymal_c_B" xmlns:xacro="http://www.ros.org/wiki/xacro">
   <!-- Arguments -->
-  <xacro:arg name="suffix"                        default="B"/>
+  <xacro:arg name="suffix_B"                        default="B"/>
   <xacro:arg name="simulation"                    default="true"/>
   <xacro:arg name="perfect_sensors"               default="true"/>

File: src/anymal_c_twins/urdf/anymal_c_Renamable_child.urdf.xacro (robot description, xacro)
@@ -2,7 +2,7 @@
 <!-- This file contains the description of the ANYmal robot. -->
 <robot name="anymal_c_B" xmlns:xacro="http://www.ros.org/wiki/xacro">
-  <xacro:macro name="anymal_c_macro" params="suffix parent_link">
+  <xacro:macro name="anymal_c_macro" params="suffix parent_link xyz rpy">
     <!-- Arguments -->
-    <xacro:arg name="suffix"                        default="${suffix}"/>
+    <!--xacro:arg name="suffix"                        default="${suffix}"/-->
     <xacro:arg name="simulation"                    default="true"/>
     <xacro:arg name="perfect_sensors"               default="true"/>
@@ -47,5 +47,5 @@
     <xacro:if value="${version_ == 'c100'}">
       <xacro:include filename="$(find anymal_c_twins)/urdf/base/base_3_1_1_macro.urdf.xacro"/>
-      <xacro:base suffix="$(arg suffix)"
+      <xacro:base suffix="${suffix}"
                   fix_base="$(arg fix_base)"
                   simulate_depth_camera="$(arg simulate_depth_camera)"
@@ -72,5 +72,5 @@
         <parent link="${parent_link}" />
         <child link="base_${suffix}" />
-        <origin xyz="0.6 0 -0.35" rpy="0 0 1.57079633"/>
+        <origin xyz="${xyz}" rpy="${rpy}"/>
 		  </joint>
     </xacro:if>
@@ -111,12 +111,12 @@
       <xacro:include filename="$(find anymal_c_twins)/urdf/leg/leg_3_1_1_macro.urdf.xacro"/>
     </xacro:if>
-    <xacro:leg leg="LF" suffix="$(arg suffix)"/>
-    <xacro:leg leg="RF" suffix="$(arg suffix)"/>
-    <xacro:leg leg="LH" suffix="$(arg suffix)"/>
-    <xacro:leg leg="RH" suffix="$(arg suffix)"/>
+    <xacro:leg leg="LF" suffix="${suffix}"/>
+    <xacro:leg leg="RF" suffix="${suffix}"/>
+    <xacro:leg leg="LH" suffix="${suffix}"/>
+    <xacro:leg leg="RH" suffix="${suffix}"/>
     <!-- Custom payload -->
     <xacro:if value="$(arg enable_custom_payload)">
       <xacro:include filename="$(arg custom_payload_description)"/>
-      <xacro:custom_payload parent="base_$(arg suffix)" />
+      <xacro:custom_payload parent="base_${suffix}" />
     </xacro:if>
     <!-- Inspection payload -->
@@ -124,5 +124,5 @@
     <xacro:if value="$(arg enable_inspection_payload)">
       <xacro:include filename="$(find inspection_payload_description)/urdf/inspection_payload_odrive.urdf.xacro"/>
-      <xacro:inspection_payload name="inspection_payload" parent="base_$(arg suffix)" version="${inspection_payload_version_}">
+      <xacro:inspection_payload name="inspection_payload" parent="base_${suffix}" version="${inspection_payload_version_}">
         <origin xyz="0.116 0.0 0.090" rpy="0 0 0"/>
       </xacro:inspection_payload>

File: src/anytwin_urdf_development/urdf/anymal_c.urdf.xacro (robot description, xacro)
@@ -2,5 +2,5 @@
 <robot name="anymal_c" xmlns:xacro="http://www.ros.org/wiki/xacro">
     <xacro:include filename="$(find anymal_c_twins)/urdf/anymal_c_Renamable.urdf.xacro"/>
+    <xacro:anymal_c_macro suffix='A'/>
     <xacro:anymal_c_macro suffix='B'/>
-    <!--xacro:anymal_c_macro suffix='B'/-->
 </robot>

File: src/anytwin_urdf_development/urdf/anytwin_c.urdf.xacro (robot description, xacro)
@@ -1,18 +1,8 @@
 <?xml version="1.0"?>
 <robot name="anytwins" xmlns:xacro="http://www.ros.org/wiki/xacro">
-<!--include macro to load anymal_c versions A and B-->
-    <!--xacro:include filename="$(find anytwin_urdf_development)/urdf/anymal_c.urdf.xacro"/-->
-    <xacro:arg name="suffix_one" default="A"/>
-    <xacro:arg name="suffix_two" default="B"/>
-    <!--xacro:macro name="anymal_c_macro" params="suffix">
-        <xacro:include filename="$(find anymal_c_twins)/urdf/anymal_c_${suffix}.urdf.xacro"/>
-    </xacro:macro-->
     <xacro:include filename="$(find anytwin_urdf_development)/urdf/linkage.urdf.xacro"/>
-    <!--xacro:anymal_c_macro suffix="$(arg suffix_one)"/>
-    <xacro:anymal_c_macro suffix="$(arg suffix_two)"/-->
     <xacro:include filename="$(find anymal_c_twins)/urdf/anymal_c_Renamable_child.urdf.xacro"/>
-    <!--xacro:anymal_c_macro-->
-    <xacro:anymal_c_macro suffix='A' parent_link='base_link'/>
-    <!--xacro:anymal_c_macro suffix='B' parent_link='base_link'/-->
-    <!--/xacro:anymal_c_macro-->
+    <xacro:anymal_c_macro suffix='B' parent_link='base_link' xyz="0.6 0 -0.35" rpy="0 0 1.57079633"/>
+    <!--In the following call, it doesn't use 'B' but rather 'A' from the first call again-->
+    <xacro:anymal_c_macro suffix='A' parent_link='base_link' xyz="-0.6 0 -0.35" rpy="0 0 1.57079633"/>
 </robot>
