Commit message: Make actually renamable

File: src/anymal_c_twins/urdf/base/face/face_3_1_1_macro.urdf.xacro (robot description, xacro)
@@ -1,5 +1,5 @@
 <?xml version="1.0"?>
 <robot xmlns:xacro="http://www.ros.org/wiki/xacro">
-  <xacro:macro name="face" params="suffix:='A' face simulate_depth_camera:=false simulate_wide_angle_camera:=false depth_camera_pitch:=30 depth_camera_roll:=0">
+  <xacro:macro name="face" params="suffix face simulate_depth_camera:=false simulate_wide_angle_camera:=false depth_camera_pitch:=30 depth_camera_roll:=0">
     <xacro:property name="B_r_BBf_x"        value="0.41450"/> <!--  [m] -->
     <xacro:property name="B_r_BBf_z"        value="0.00700"/> <!--  [m] -->

File: src/anytwin_urdf_development/urdf/anymal_c.urdf.xacro (robot description, xacro)
@@ -1,7 +1,5 @@
 <?xml version="1.0"?>
 <robot name="anymal_c" xmlns:xacro="http://www.ros.org/wiki/xacro">
-    <xacro:macro name="anymal_c_macro" params="suffix:='A'">
-        <xacro:include filename="$(find anymal_c_twins)/urdf/anymal_c_${suffix}.urdf.xacro"/>
-    </xacro:macro>
-    <xacro:anymal_c_macro suffix='B'/>
+    <xacro:include filename="$(find anymal_c_twins)/urdf/anymal_c_Renamable.urdf.xacro"/>
+    <xacro:anymal_c_macro suffix='A'/>
 </robot>

File: src/anytwin_urdf_development/urdf/anytwin_c.urdf.xacro (robot description, xacro)
@@ -1,4 +1,4 @@
 <?xml version="1.0"?>
-<robot name="anymal_c" xmlns:xacro="http://www.ros.org/wiki/xacro">
+<robot name="anytwins" xmlns:xacro="http://www.ros.org/wiki/xacro">
 <!--include macro to load anymal_c versions A and B-->
     <!--xacro:include filename="$(find anytwin_urdf_development)/urdf/anymal_c.urdf.xacro"/-->
@@ -8,4 +8,5 @@
         <xacro:include filename="$(find anymal_c_twins)/urdf/anymal_c_${suffix}.urdf.xacro"/>
     </xacro:macro>
+    <xacro:include filename="$(find anymal_c_twins)/urdf/linkage.urdf.xacro"/>
     <!--xacro:anymal_c_macro suffix="$(arg suffix_one)"/>
     <xacro:anymal_c_macro suffix="$(arg suffix_two)"/-->
